File: 01_DESIGN/BEE-1012_PAY-IF_V110/CAN_PHY.kicad_sch (KiCad schematic)
At the start: 16 parts, among them U30 SN65HVD230DR, U31 SN65HVD230DR

Commit message: Done Layout
Connections:
- net CAN_H_AX100U renamed CAN_AX100U_P
- net CAN_H_main renamed CAN_main_P
- net CAN_L_AX100U renamed CAN_AX100U_N
- net CAN_L_main renamed CAN_main_N
Changed lines of the file:
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@@
 		)
 	)
-	(global_label "CAN_L_main"
+	(global_label "CAN_main_N"
 		(shape bidirectional)
 		(at 158.75 52.07 0)
@@
 		)
 		(property "Intersheetrefs" "${INTERSHEET_REFS}"
-			(at 174.095 52.07 0)
+			(at 174.3974 52.07 0)
 			(hide yes)
 			(show_name no)
@@
 		)
 	)
-	(global_label "CAN_H_AX100U"
+	(global_label "CAN_AX100U_P"
 		(shape bidirectional)
 		(at 158.75 125.73 0)
@@
 		)
 		(property "Intersheetrefs" "${INTERSHEET_REFS}"
-			(at 177.0584 125.73 0)
+			(at 176.9979 125.73 0)
 			(hide yes)
 			(show_name no)
@@
 		)
 	)
-	(global_label "CAN_H_main"
+	(global_label "CAN_main_P"
 		(shape bidirectional)
 		(at 158.75 46.99 0)
@@
 		)
 		(property "Intersheetrefs" "${INTERSHEET_REFS}"
-			(at 174.3974 46.99 0)
+			(at 174.3369 46.99 0)
 			(hide yes)
 			(show_name no)
@@
 		)
 	)
-	(global_label "CAN_L_AX100U"
+	(global_label "CAN_AX100U_N"
 		(shape bidirectional)
 		(at 158.75 130.81 0)
@@
 		)
 		(property "Intersheetrefs" "${INTERSHEET_REFS}"
-			(at 176.756 130.81 0)
+			(at 177.0584 130.81 0)
 			(hide yes)
 			(show_name no)
