File: 01_DESIGN/BEE-1012_PAY-IF_V110/CONNECTOR_INTERFACE.kicad_sch (KiCad schematic)
At the start: 60 parts, among them J10 5040500991, J11 FSI-110-03-G-D-AD, J12 TLE-110-01-G-DV-A-TR, J13 5040500691, J14 5040500691, J5 5040500691, J6 ESQ-126-14-G-D, J7 ESQ-126-14-G-D, J8 5040500491, J9 5040500991

Commit message: Done Layout
Connections:
- net CAN_H_AX100U renamed CAN_AX100U_P
- net CAN_H_main renamed CAN_main_P
- net CAN_L_AX100U renamed CAN_AX100U_N
- net CAN_L_main renamed CAN_main_N
Changed lines of the file:
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@@
 		)
 	)
-	(global_label "CAN_H_AX100U"
+	(global_label "CAN_AX100U_P"
 		(shape bidirectional)
 		(at 209.55 29.21 180)
@@
 		)
 		(property "Intersheetrefs" "${INTERSHEET_REFS}"
-			(at 191.2416 29.21 0)
+			(at 191.3021 29.21 0)
 			(hide yes)
 			(show_name no)
@@
 		)
 	)
-	(global_label "CAN_L_AX100U"
+	(global_label "CAN_AX100U_N"
 		(shape bidirectional)
 		(at 209.55 26.67 180)
@@
 		)
 		(property "Intersheetrefs" "${INTERSHEET_REFS}"
-			(at 191.544 26.67 0)
+			(at 191.2416 26.67 0)
 			(hide yes)
 			(show_name no)
@@
 		)
 	)
-	(global_label "CAN_H_AX100U"
+	(global_label "CAN_AX100U_P"
 		(shape bidirectional)
 		(at 265.43 146.05 180)
@@
 		)
 		(property "Intersheetrefs" "${INTERSHEET_REFS}"
-			(at 247.1216 146.05 0)
+			(at 247.1821 146.05 0)
 			(hide yes)
 			(show_name no)
@@
 		)
 	)
-	(global_label "CAN_L_main"
+	(global_label "CAN_main_N"
 		(shape bidirectional)
 		(at 209.55 33.02 180)
@@
 		)
 		(property "Intersheetrefs" "${INTERSHEET_REFS}"
-			(at 194.205 33.02 0)
-			(hide yes)
-			(show_name no)
-			(do_not_autoplace no)
-			(effects
-				(font
-					(size 1.27 1.27)
-				)
-				(justify right)
-			)
-		)
-	)
-	(global_label "CAN_H_main"
+			(at 193.9026 33.02 0)
+			(hide yes)
+			(show_name no)
+			(do_not_autoplace no)
+			(effects
+				(font
+					(size 1.27 1.27)
+				)
+				(justify right)
+			)
+		)
+	)
+	(global_label "CAN_main_P"
 		(shape bidirectional)
 		(at 209.55 35.56 180)
@@
 		)
 		(property "Intersheetrefs" "${INTERSHEET_REFS}"
-			(at 193.9026 35.56 0)
+			(at 193.9631 35.56 0)
 			(hide yes)
 			(show_name no)
@@
 		)
 	)
-	(global_label "CAN_L_AX100U"
+	(global_label "CAN_AX100U_N"
 		(shape bidirectional)
 		(at 318.77 146.05 0)
@@
 		)
 		(property "Intersheetrefs" "${INTERSHEET_REFS}"
-			(at 336.776 146.05 0)
-			(hide yes)
-			(show_name no)
+			(at 337.0784 146.05 0)
+			(hide yes)
+			(show_name no)
