File: 01_DESIGN/BEE-1012_PAY-IF_V110/SAMA7G54_PIO.kicad_sch (KiCad schematic)
At the start: 120 parts, among them J15 Header 8x1, U8 SAMA7G54

Commit message: Done Layout
Connections:
- net NRST renamed nRST
Changed lines of the file:
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@@
 		)
 	)
-	(global_label "NRST"
+	(global_label "nRST"
 		(shape output)
 		(at 342.9 114.3 0)
@@
 		)
 		(property "Intersheetrefs" "${INTERSHEET_REFS}"
-			(at 350.6628 114.3 0)
+			(at 350.4813 114.3 0)
 			(hide yes)
 			(show_name no)
