File: 01_DESIGN/BEE-1012_PAY-IF_V110/TEMP.kicad_sch (KiCad schematic)
At the start: 31 parts, among them J19 5040500891, U21 TC1047AVNBTR, U22 OPA2340, U23 OPA2340

Commit message: Done Layout
Connections:
- net at R282.1, U22.7: now also U22.6 (-); no longer U22.5 (+)
- net at C167.2, R283.2: now also U22.5 (+); no longer U22.6 (-)
- net at C173.2, R289.2: now also U23.5 (+); no longer U23.6 (-)
- net at R288.1, U23.7: now also U23.6 (-); no longer U23.5 (+)
Changed lines of the file:
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@@
 	)
 	(junction
-		(at 137.16 195.58)
-		(diameter 0)
-		(color 0 0 0 0)
-	)
-	(junction
-		(at 137.16 132.08)
-		(diameter 0)
-		(color 0 0 0 0)
-	)
-	(junction
 		(at 106.68 167.64)
 		(diameter 0)
@@
 	)
 	(junction
-		(at 106.68 198.12)
+		(at 54.61 172.72)
 		(diameter 0)
 		(color 0 0 0 0)
 	)
 	(junction
-		(at 54.61 172.72)
+		(at 148.59 33.02)
 		(diameter 0)
 		(color 0 0 0 0)
 	)
 	(junction
-		(at 148.59 33.02)
+		(at 137.16 132.08)
 		(diameter 0)
 		(color 0 0 0 0)
@@
 	)
 	(junction
+		(at 106.68 198.12)
+		(diameter 0)
+		(color 0 0 0 0)
+	)
+	(junction
 		(at 154.94 132.08)
 		(diameter 0)
@@
 	)
 	(junction
-		(at 154.94 195.58)
+		(at 106.68 134.62)
 		(diameter 0)
 		(color 0 0 0 0)
 	)
 	(junction
-		(at 106.68 134.62)
+		(at 154.94 195.58)
 		(diameter 0)
 		(color 0 0 0 0)
@@
 	)
 	(junction
+		(at 137.16 195.58)
+		(diameter 0)
+		(color 0 0 0 0)
+	)
+	(junction
 		(at 91.44 104.14)
 		(diameter 0)
@@
 	(wire
 		(pts
-			(xy 118.11 198.12) (xy 106.68 198.12)
+			(xy 106.68 205.74) (xy 106.68 208.28)
 		)
 		(stroke
@@
 	(wire
 		(pts
-			(xy 106.68 205.74) (xy 106.68 208.28)
+			(xy 114.3 88.9) (xy 137.16 88.9)
 		)
 		(stroke
@@
 	(wire
 		(pts
-			(xy 114.3 88.9) (xy 137.16 88.9)
+			(xy 50.8 49.53) (xy 54.61 49.53)
 		)
 		(stroke
@@
 	(wire
 		(pts
-			(xy 50.8 49.53) (xy 54.61 49.53)
+			(xy 91.44 134.62) (xy 95.25 134.62)
 		)
 		(stroke
@@
 	(wire
 		(pts
-			(xy 91.44 134.62) (xy 95.25 134.62)
+			(xy 114.3 119.38) (xy 137.16 119.38)
 		)
 		(stroke
@@
 	(wire
 		(pts
-			(xy 114.3 119.38) (xy 137.16 119.38)
+			(xy 133.35 195.58) (xy 137.16 195.58)
+		)
+		(stroke
+			(width 0)
+			(type default)
+		)
+	)
+	(wire
+		(pts
+			(xy 106.68 134.62) (xy 118.11 134.62)
 		)
 		(stroke
@@
 	(wire
 		(pts
-			(xy 137.16 119.38) (xy 137.16 132.08)
+			(xy 133.35 132.08) (xy 137.16 132.08)
 		)
 		(stroke
@@
 	(wire
 		(pts
-			(xy 154.94 132.08) (xy 154.94 135.89)
+			(xy 137.16 119.38) (xy 137.16 132.08)
 		)
 		(stroke
@@
 	(wire
 		(pts
-			(xy 91.44 104.14) (xy 95.25 104.14)
+			(xy 154.94 132.08) (xy 154.94 135.89)
 		)
 		(stroke
@@
 	(wire
 		(pts
-			(xy 152.4 48.26) (xy 148.59 48.26)
+			(xy 91.44 104.14) (xy 95.25 104.14)
 		)
 		(stroke
@@
 	(wire
 		(pts
-			(xy 151.13 132.08) (xy 154.94 132.08)
+			(xy 152.4 48.26) (xy 148.59 48.26)
 		)
 		(stroke
@@
 	(wire
 		(pts
-			(xy 151.13 165.1) (xy 154.94 165.1)
+			(xy 151.13 132.08) (xy 154.94 132.08)
 		)
 		(stroke
@@
 	(wire
 		(pts
-			(xy 106.68 142.24) (xy 106.68 144.78)
+			(xy 151.13 165.1) (xy 154.94 165.1)
 		)
 		(stroke
@@
 	(wire
 		(pts
-			(xy 91.44 135.89) (xy 91.44 134.62)
+			(xy 106.68 142.24) (xy 106.68 144.78)
 		)
 		(stroke
@@
 	(wire
 		(pts
-			(xy 118.11 193.04) (xy 114.3 193.04)
+			(xy 91.44 135.89) (xy 91.44 134.62)
 		)
 		(stroke
@@
 	(wire
 		(pts
-			(xy 133.35 195.58) (xy 137.16 195.58)
-		)
-		(stroke
-			(width 0)
-			(type default)
-		)
-	)
-	(wire
-		(pts
 			(xy 137.16 88.9) (xy 137.16 101.6)
 		)
@@
 	(wire
 		(pts
-			(xy 118.11 134.62) (xy 106.68 134.62)
+			(xy 154.94 132.08) (xy 170.18 132.08)
 		)
 		(stroke
@@
 	(wire
 		(pts
-			(xy 154.94 132.08) (xy 170.18 132.08)
+			(xy 82.55 198.12) (xy 91.44 198.12)
 		)
 		(stroke
@@
 	(wire
 		(pts
-			(xy 82.55 198.12) (xy 91.44 198.12)
+			(xy 118.11 99.06) (xy 114.3 99.06)
 		)
 		(stroke
@@
 	(wire
 		(pts
-			(xy 118.11 99.06) (xy 114.3 99.06)
+			(xy 114.3 129.54) (xy 118.11 129.54)
 		)
 		(stroke
@@
 	(wire
 		(pts
-			(xy 118.11 129.54) (xy 114.3 129.54)
-		)
-		(stroke
-			(width 0)
-			(type default)
-		)
-	)
-	(wire
-		(pts
 			(xy 25.4 52.07) (xy 25.4 58.42)
 		)
@@
 	(wire
 		(pts
-			(xy 137.16 182.88) (xy 137.16 195.58)
+			(xy 106.68 198.12) (xy 118.11 198.12)
 		)
 		(stroke
@@
 	(wire
 		(pts
-			(xy 148.59 58.42) (xy 148.59 60.96)
+			(xy 114.3 193.04) (xy 118.11 193.04)
 		)
 		(stroke
@@
 	(wire
 		(pts
-			(xy 146.05 50.8) (xy 152.4 50.8)
+			(xy 137.16 182.88) (xy 137.16 195.58)
 		)
 		(stroke
@@
 	(wire
 		(pts
-			(xy 43.18 40.64) (xy 43.18 41.91)
+			(xy 148.59 58.42) (xy 148.59 60.96)
 		)
 		(stroke
@@
 	(wire
 		(pts
-			(xy 154.94 140.97) (xy 154.94 144.78)
+			(xy 146.05 50.8) (xy 152.4 50.8)
 		)
 		(stroke
@@
 	(wire
 		(pts
-			(xy 39.37 109.22) (xy 39.37 115.57)
+			(xy 43.18 40.64) (xy 43.18 41.91)
 		)
 		(stroke
@@
 	(wire
 		(pts
-			(xy 133.35 132.08) (xy 137.16 132.08)
+			(xy 154.94 140.97) (xy 154.94 144.78)
+		)
+		(stroke
+			(width 0)
+			(type default)
+		)
+	)
+	(wire
+		(pts
+			(xy 39.37 109.22) (xy 39.37 115.57)
 		)
 		(stroke
@@
 		(lib_id "Amplifier_Operational:OPA2340")
 		(at 125.73 132.08 0)
+		(mirror x)
 		(unit 2)
 		(body_style 1)
@@
 		(in_pos_files yes)
 		(dnp no)
-		(fields_autoplaced yes)
 		(property "Reference" "U22"
 			(at 125.73 121.92 0)
@@
 		(lib_id "Amplifier_Operational:OPA2340")
 		(at 125.73 195.58 0)
+		(mirror x)
 		(unit 2)
 		(body_style 1)
@@
 		(in_pos_files yes)
 		(dnp no)
-		(fields_autoplaced yes)
 		(property "Reference" "U23"
 			(at 125.73 185.42 0)
