File: 01_DESIGN/BEE-1012_PAY-IF_V110/WATCHDOG.kicad_sch (KiCad schematic)
At the start: 8 parts, among them U25 TPL5010DDCR

Commit message: Done Layout
Connections:
- net NRST renamed nRST
Changed lines of the file:
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@@
 		)
 	)
-	(global_label "NRST"
+	(global_label "nRST"
 		(shape output)
 		(at 124.46 38.1 0)
@@
 		)
 		(property "Intersheetrefs" "${INTERSHEET_REFS}"
-			(at 132.2228 38.1 0)
+			(at 132.0413 38.1 0)
 			(hide yes)
 			(show_name no)
